File: cq2-kicad/cpci-connector.kicad_sch (KiCad schematic)
At the start: 68 parts, among them J2 HM2 110 TypeA

Commit message: drc checked before panalization
Parts:
- removed FID10, FID11, FID12, FID7, FID8, FID9: Fiducial 1.0, 1-special:various-9, symbol ci4rail-database:various/9
Other:
- note removed: "2024-07-03"
- note removed: "A"
- note removed: "CompactPCi Connector"
- note removed: "M.Schmitz"
- note removed: "tbd"
- title: (none) -> CQ2
