File: cq2-kicad/esp32s2.kicad_sch (KiCad schematic)
At the start: 37 parts, among them U15 APX803L20-31SA-7, U16 ESP32-S2FH4, U17 IS25LP032D, U18 IS25LP032D, X3 40 MHz

Commit message: drc checked before panalization
Parts:
- C108, C109: now not fitted
Other:
- note removed: "Manfred Schmitz"
- title: (none) -> CQ2

Commit message: Production documents created
Parts:
- R167, R168, R169, R170, R171: Value2 100 ppm -> (none); Value3 62.5 mW -> (none); Value4 50 V -> (none)
Changed lines of the file:
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@@
 	(title_block
 		(title "CQ2")
-		(date "2024-07-31")
+		(date "2024-08-03")
 		(rev "0")
 		(comment 2 "Manfred Schmitz")
@@
 			)
 		)
-		(property "Value2" "100 ppm"
+		(property "Value2" ""
 			(at 179.07 106.68 0)
 			(effects
@@
 			)
 		)
-		(property "Value3" "62.5 mW"
+		(property "Value3" ""
 			(at 179.07 106.68 0)
 			(effects
@@
 			)
 		)
-		(property "Value4" "50 V"
+		(property "Value4" ""
 			(at 179.07 106.68 0)
 			(effects
@@
 			)
 		)
-		(property "Value2" "100 ppm"
+		(property "Value2" ""
 			(at 179.07 101.6 0)
 			(effects
@@
 			)
 		)
-		(property "Value3" "62.5 mW"
+		(property "Value3" ""
 			(at 179.07 101.6 0)
 			(effects
@@
 			)
 		)
-		(property "Value4" "50 V"
+		(property "Value4" ""
 			(at 179.07 101.6 0)
 			(effects
@@
 			)
 		)
-		(property "Value2" "100 ppm"
+		(property "Value2" ""
 			(at 179.07 104.14 0)
 			(effects
@@
 			)
 		)
-		(property "Value3" "62.5 mW"
+		(property "Value3" ""
 			(at 179.07 104.14 0)
 			(effects
@@
 			)
 		)
-		(property "Value4" "50 V"
+		(property "Value4" ""
 			(at 179.07 104.14 0)
 			(effects
@@
 			)
 		)
-		(property "Value2" "100 ppm"
+		(property "Value2" ""
 			(at 179.07 114.3 0)
 			(effects
@@
 			)
 		)
-		(property "Value3" "62.5 mW"
+		(property "Value3" ""
 			(at 179.07 114.3 0)
 			(effects
@@
 			)
 		)
-		(property "Value4" "50 V"
+		(property "Value4" ""
 			(at 179.07 114.3 0)
 			(effects
@@
 			)
 		)
-		(property "Value2" "100 ppm"
+		(property "Value2" ""
 			(at 179.07 111.76 0)
 			(effects
@@
 			)
 		)
-		(property "Value3" "62.5 mW"
+		(property "Value3" ""
 			(at 179.07 111.76 0)
 			(effects
@@
 			)
 		)
-		(property "Value4" "50 V"
+		(property "Value4" ""
 			(at 179.07 111.76 0)
 			(effects
