File: cq2-kicad/output-switch.kicad_sch (KiCad schematic)
At the start: 9 parts, among them U39 TLP175A, U40 TLP3545A, U41 TLP175A

Commit message: drc checked before panalization
Other:
- note removed: "2024-07-03"
- note removed: "A"
- note removed: "Controlled PSU"
- note removed: "M.Schmitz"
- note removed: "tbd"
Changed lines of the file:
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@@
 	(title_block
 		(title "CQ2")
-		(date "2024-07-17")
+		(date "2024-07-31")
 		(rev "0")
+		(comment 1 "Output Switch")
+		(comment 2 "Manfred Schmitz")
+		(comment 3 "tbd")
+		(comment 4 "2024-07-03")
+		(comment 5 "tbd")
+		(comment 6 "A")
 	)

Commit message: Production documents created
Parts:
- U39, U41: Lifecycle review pending CQ2 -> ERP1 pending CQ2; Outline (none) -> SMT MFSOP6-4_4.4x3.6mm
- U40: Lifecycle review pending CQ2 -> ERP1 pending CQ2; Outline (none) -> SMT SMDIP-6_W7.62mm
Changed lines of the file:
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@@
 	(title_block
 		(title "CQ2")
-		(date "2024-07-31")
+		(date "2024-08-03")
 		(rev "0")
 		(comment 1 "Output Switch")
