File: cq2-kicad/unisolated_io.kicad_sch (KiCad schematic)
At the start: 16 parts, among them U64 PCAL9722

Commit message: drc checked before panalization
Other:
- note removed: "2024-01-12"
- note removed: "A"
- note removed: "M.Schmitz"
- note removed: "S.Poß"
- note removed: "SPI based GPIO Extension"
- note removed: "tbd"
Changed lines of the file:
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@@
 	(title_block
 		(title "CQ2")
-		(date "2024-07-17")
+		(date "2024-07-31")
 		(rev "0")
+		(comment 1 "SPI based GPIO Extension")
+		(comment 2 "Manfred Schmitz")
+		(comment 3 "tbd")
+		(comment 4 "2024-07-03")
+		(comment 5 "tbd")
+		(comment 6 "A")
 	)
 	(junction
@@
 		)
 	)
-	(text "tbd"
-		(exclude_from_sim no)
-		(at 238.125 193.675 0)
-		(effects
-			(font
-				(size 1.27 1.27)
-			)
-			(justify left bottom)
-		)
-	)
-	(text "2024-01-12"
-		(exclude_from_sim no)
-		(at 238.125 191.135 0)
-		(effects
-			(font
-				(size 1.27 1.27)
-			)
-			(justify left bottom)
-		)
-	)
-	(text "S.Poß"
-		(exclude_from_sim no)
-		(at 192.405 193.675 0)
-		(effects
-			(font
-				(size 1.27 1.27)
-			)
-			(justify left bottom)
-		)
-	)
-	(text "SPI based GPIO Extension"
-		(exclude_from_sim no)
-		(at 192.405 187.325 0)
-		(effects
-			(font
-				(size 1.27 1.27)
-			)
-			(justify left bottom)
-		)
-	)
-	(text "A"
-		(exclude_from_sim no)
-		(at 270.51 192.405 0)
-		(effects
-			(font
-				(size 1.4986 1.4986)
-			)
-			(justify left bottom)
-		)
-	)
-	(text "M.Schmitz"
-		(exclude_from_sim no)
-		(at 192.405 191.135 0)
-		(effects
-			(font
-				(size 1.27 1.27)
-			)
-			(justify left bottom)
-		)
-	)
 	(label "GND"
 		(at 74.93 125.73 0)
@@
 			)
 		)
-		(property "Lifecyle" ""
-			(at 182.88 72.39 0)
-			(effects
-				(font
-					(size 1.27 1.27)
-				)
-				(hide yes)
-			)
-		)
 		(pin "2"
 		)
@@
 			)
 		)
-		(property "Lifecyle" ""
-			(at 195.58 93.98 0)
-			(effects
-				(font
-					(size 1.27 1.27)
-				)
-				(hide yes)
-			)
-		)
 		(pin "4"
 		)
@@
 			)
 		)
-		(property "Lifecyle" ""
-			(at 182.88 101.6 0)
-			(effects
-				(font
-					(size 1.27 1.27)
-				)
-				(hide yes)
-			)
-		)
 		(pin "2"
 		)
@@
 			)
 		)
-		(property "Lifecyle" ""
-			(at 195.58 35.56 0)
-			(effects
-				(font
-					(size 1.27 1.27)
-				)
-				(hide yes)
-			)
-		)
 		(pin "4"
 		)
@@
 			)
 		)
-		(property "Lifecyle" ""
-			(at 182.88 130.81 0)
-			(effects
-				(font
-					(size 1.27 1.27)
-				)
-				(hide yes)
-			)
-		)
 		(pin "2"
 		)
@@
 			)
 		)
-		(property "Lifecyle" ""
-			(at 182.88 43.18 0)
-			(effects
-				(font
-					(size 1.27 1.27)
-				)
-				(hide yes)
-			)
-		)
 		(pin "2"
 		)
@@
 			)
 		)
-		(property "Lifecyle" ""
-			(at 195.58 64.77 0)
-			(effects
-				(font
-					(size 1.27 1.27)
-				)
-				(hide yes)
-			)
-		)
 		(pin "4"
 		)
@@
 			)
 		)
-		(property "Lifecyle" ""
-			(at 182.88 74.93 0)
-			(effects
-				(font
-					(size 1.27 1.27)
-				)
-				(hide yes)
-			)
-		)
 		(pin "1"
 		)
@@
 			)
 		)
-		(property "Lifecyle" ""
-			(at 182.88 133.35 0)
-			(effects
-				(font
-					(size 1.27 1.27)
-				)
-				(hide yes)
-			)
-		)
 		(pin "1"
 		)
@@
 			)
 		)
-		(property "Lifecyle" ""
-			(at 195.58 123.19 0)
-			(effects
-				(font
-					(size 1.27 1.27)
-				)
-				(hide yes)
-			)
-		)
 		(pin "4"
 		)
@@
 			)
 		)
-		(property "Lifecyle" ""
-			(at 182.88 104.14 0)
-			(effects
-				(font
-					(size 1.27 1.27)
-				)
-				(hide yes)
-			)
-		)
 		(pin "1"
 		)
@@
 			(at 182.88 45.72 0)
 			(effects
-				(font
-					(size 1.27 1.27)
-				)
-				(hide yes)
-			)
-		)
-		(property "Lifecyle" ""
-			(at 182.88 45.72 0)
-			(effects

Commit message: Production documents created
Parts:
- H14: Outline MM 15.7x11.3X4.9 -> MMT 15.7x11.3X4.9
Changed lines of the file:
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@@
 	(title_block
 		(title "CQ2")
-		(date "2024-07-31")
+		(date "2024-08-03")
 		(rev "0")
 		(comment 1 "SPI based GPIO Extension")
@@
 			)
 		)
-		(property "Outline" "MM 15.7x11.3X4.9"
+		(property "Outline" "MMT 15.7x11.3X4.9"
 			(at 229.87 143.51 0)
 			(effects

Commit message: cq2 adapter in work
Changed lines of the file:
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@@
 (kicad_sch
-	(version 20231120)
+	(version 20250114)
 	(generator "eeschema")
-	(generator_version "8.0")
+	(generator_version "9.0")
 	(paper "A4")
 	(title_block
@@
 	(label "GND"
 		(at 74.93 125.73 0)
-		(fields_autoplaced yes)
 		(effects
 			(font
@@
 	(label "+3V3"
 		(at 173.99 113.03 0)
-		(fields_autoplaced yes)
 		(effects
 			(font
@@
 	(label "+3V3"
 		(at 173.99 54.61 0)
-		(fields_autoplaced yes)
 		(effects
 			(font
@@
 	(label "GND"
 		(at 74.93 82.55 0)
-		(fields_autoplaced yes)
 		(effects
 			(font
@@
 	(label "+3V3"
 		(at 173.99 83.82 0)
-		(fields_autoplaced yes)
 		(effects
 			(font
@@
 	(label "+3V3"
 		(at 173.99 25.4 0)
-		(fields_autoplaced yes)
 		(effects
 			(font
@@
 	(label "GND"
 		(at 74.93 123.19 0)
-		(fields_autoplaced yes)
 		(effects
 			(font
@@
 	(label "+3V3"
 		(at 121.92 62.23 180)
-		(fields_autoplaced yes)
 		(effects
 			(font
@@
 	(label "+3V3"
 		(at 74.93 62.23 0)
-		(fields_autoplaced yes)
 		(effects
 			(font
@@
 		(shape input)
 		(at 62.23 118.11 180)
-		(fields_autoplaced yes)
 		(effects
 			(font
@@
 		(shape input)
 		(at 62.23 95.25 180)
-		(fields_autoplaced yes)
 		(effects
 			(font
@@
 		(shape output)
 		(at 129.54 113.03 0)
-		(fields_autoplaced yes)
 		(effects
 			(font
@@
 		(shape input)
 		(at 62.23 90.17 180)
-		(fields_autoplaced yes)
 		(effects
 			(font
@@
 		(shape input)
 		(at 93.98 137.16 180)
-		(fields_autoplaced yes)
 		(effects
 			(font
@@
 		(shape input)
 		(at 62.23 92.71 180)
-		(fields_autoplaced yes)
 		(effects
 			(font
@@
 		(shape output)
 		(at 62.23 97.79 180)
-		(fields_autoplaced yes)
 		(effects
 			(font
@@
 		(shape input)
 		(at 93.98 147.32 180)
-		(fields_autoplaced yes)
-		(effects
-			(font
+		(effects
+			(font
